Commit message: limited horizontal FOV

File: ouster_os1/urdf/os1_32.urdf.xacro (robot description, xacro)
@@ -4,4 +4,5 @@
   <xacro:property name="PI" value="3.1415926535897931"/>
   <xacro:property name="PI2" value="1.570796327"/>
+  <xacro:property name="PI34" value="2.35619449"/>
   <xacro:macro name="os1_32" params="*origin parent:=base name:=ouster reduced:=true prefix:=/os1_cloud_node hz:=10 samples:=512 min_range:=0.8 max_range:=100 noise:=0.008 min_angle_v:=-16.6 max_angle_v:=16.6 gpu:=false">
     <xacro:property name="file_visual" value="SensorAssemblyOS1"/>
@@ -86,6 +87,6 @@
               <samples>${samples}</samples>
               <resolution>1</resolution>
-              <min_angle>-${PI}</min_angle>
-              <max_angle>${PI}</max_angle>
+              <min_angle>-${PI34}</min_angle>
+              <max_angle>${PI34}</max_angle>
             </horizontal>
           </scan>
